Commit message: clean up

File: urdfs/psyonic_panda.urdf (robot description, URDF)
Before this commit: robot psyonic_panda, 26 links, 25 joints
Links:
- link hand_base: geometry collision mesh filename=psyonic/models/wristmesh.STL; visual mesh filename=psyonic/models/wristmesh.STL

Commit message: Update psyonic_panda.urdf
Fixed Psyonic hand collision issue

File: urdfs/psyonic_panda.urdf (robot description, URDF)
Before this commit: robot psyonic_panda, 26 links, 25 joints
Links:
- link index_L1: geometry collision mesh filename=psyonic/models/idx-F1.STL; visual mesh filename=psyonic/models/idx-F1.STL
- link index_L2: geometry collision mesh filename=psyonic/models/idx-F2.STL; visual mesh filename=psyonic/models/idx-F2.STL
- link middle_L1: geometry collision mesh filename=psyonic/models/idx-F1.STL; visual mesh filename=psyonic/models/idx-F1.STL
- link middle_L2: geometry collision mesh filename=psyonic/models/idx-F2.STL; visual mesh filename=psyonic/models/idx-F2.STL
- link pinky_L1: geometry collision mesh filename=psyonic/models/idx-F1.STL; visual mesh filename=psyonic/models/idx-F1.STL
- link pinky_L2: geometry collision mesh filename=psyonic/models/idx-F2.STL; visual mesh filename=psyonic/models/idx-F2.STL
- link ring_L1: geometry collision mesh filename=psyonic/models/idx-F1.STL; visual mesh filename=psyonic/models/idx-F1.STL
- link ring_L2: geometry collision mesh filename=psyonic/models/idx-F2.STL; visual mesh filename=psyonic/models/idx-F2.STL
- link thumb_L1: geometry collision mesh filename=psyonic/models/thumb-F1-MIR.STL; visual mesh filename=psyonic/models/thumb-F1-MIR.STL
- link thumb_L2: geometry collision mesh filename=psyonic/models/thumb-F2.STL; visual mesh filename=psyonic/models/thumb-F2.STL
- link thumb_base: geometry collision mesh filename=psyonic/models/FB_palm_ref_MIR.STL; visual mesh filename=psyonic/models/FB_palm_ref_MIR.STL
